Commit message: add spring joint and modify PID param

File: urdf/robot.xacro (robot description, xacro)
@@ -26,11 +26,15 @@
   <xacro:property name="down_maxvel" value="${PI*3}" />
   <!--foot property-->
-  <xacro:property name="foot_mass" value="1" />
-  <xacro:property name="foot_length" value="0.3" />
+  <xacro:property name="foot_back_mass" value="0.5" />
+  <xacro:property name="foot_front_mass" value="0.5" />
+  <xacro:property name="foot_back_length" value="0.15" />
+  <xacro:property name="foot_front_length" value="0.15" />
   <xacro:property name="foot_width" value="0.15" />
   <xacro:property name="foot_height" value="0.05" />
   <xacro:property name="foot_effort" value="500" />
-  <xacro:property name="foot_lower" value="${-PI/18}" />
-  <xacro:property name="foot_upper" value="${PI/6}" />
+  <xacro:property name="foot_front_lower" value="${-PI/3}" />
+  <xacro:property name="foot_front_upper" value="0" />
+  <xacro:property name="foot_back_lower" value="${-PI/18}" />
+  <xacro:property name="foot_back_upper" value="${PI/6}" />
   <xacro:property name="foot_maxvel" value="${PI}" />
   <!-- Import all Gazebo-customization elements, including Gazebo colors -->
@@ -189,5 +193,5 @@
   <joint name="LF_joint" type="revolute">
     <limit
-       velocity="${foot_maxvel}" effort="${foot_effort}" lower="${foot_lower}" upper="${foot_upper}" />
+       velocity="${foot_maxvel}" effort="${foot_effort}" lower="${foot_back_lower}" upper="${foot_back_upper}" />
     <parent link="LD_link"/>
     <child link="LF_link"/>
@@ -197,29 +201,32 @@
   </joint>
   <link name="LF_link">
-    <collision>
-      <origin xyz="${foot_length/2-down_width/2} ${-foot_width/2} ${-foot_height/2}" rpy="0 0 0"/>
-      <geometry>
-	    <box size="${foot_length} ${foot_width} ${foot_height}"/>
-      </geometry>
-    </collision>
-    <visual>
-      <origin xyz="${foot_length/2-down_width/2} ${-foot_width/2} ${-foot_height/2}" rpy="0 0 0"/>
-      <geometry>
-	    <box size="${foot_length} ${foot_width} ${foot_height}"/>
-      </geometry>
-      <material name="orange"/>
-    </visual>
-    <inertial>
-      <origin xyz="${foot_length/2-down_width/2} ${-foot_width/2} ${-foot_height/2}" rpy="0 0 0"/>
-      <mass value="${foot_mass}"/>
-      <inertia
-	  ixx="${foot_mass / 12.0 * (foot_width*foot_width + foot_height*foot_height)}" ixy="0.0" ixz="0.0"
-	  iyy="${foot_mass / 12.0 * (foot_length*foot_length + foot_height*foot_height)}" iyz="0.0"
-	  izz="${foot_mass / 12.0 * (foot_length*foot_length + foot_width*foot_width)}"/>
+    <gazebo>
+        <self_collide>1</self_collide>
+    </gazebo>
+    <collision>
+      <origin xyz="${foot_back_length/2-down_width/2} ${-foot_width/2} ${-foot_height/2}" rpy="0 0 0"/>
+      <geometry>
+	    <box size="${foot_back_length} ${foot_width} ${foot_height}"/>
+      </geometry>
+    </collision>
+    <visual>
+      <origin xyz="${foot_back_length/2-down_width/2} ${-foot_width/2} ${-foot_height/2}" rpy="0 0 0"/>
+      <geometry>
+	    <box size="${foot_back_length} ${foot_width} ${foot_height}"/>
+      </geometry>
+      <material name="orange"/>
+    </visual>
+    <inertial>
+      <origin xyz="${foot_back_length/2-down_width/2} ${-foot_width/2} ${-foot_height/2}" rpy="0 0 0"/>
+      <mass value="${foot_back_mass}"/>
+      <inertia
+	  ixx="${foot_back_mass / 12.0 * (foot_width*foot_width + foot_height*foot_height)}" ixy="0.0" ixz="0.0"
+	  iyy="${foot_back_mass / 12.0 * (foot_back_length*foot_back_length + foot_height*foot_height)}" iyz="0.0"
+	  izz="${foot_back_mass / 12.0 * (foot_back_length*foot_back_length + foot_width*foot_width)}"/>
     </inertial>
   </link>
   <joint name="RF_joint" type="revolute">
     <limit
-       velocity="${foot_maxvel}" effort="${foot_effort}" lower="${foot_lower}" upper="${foot_upper}" />
+       velocity="${foot_maxvel}" effort="${foot_effort}" lower="${foot_back_lower}" upper="${foot_back_upper}" />
     <parent link="RD_link"/>
     <child link="RF_link"/>
@@ -230,23 +237,93 @@
   <link name="RF_link">
     <collision>
-      <origin xyz="${foot_length/2-down_width/2} ${foot_width/2} ${-foot_height/2}" rpy="0 0 0"/>
-      <geometry>
-	    <box size="${foot_length} ${foot_width} ${foot_height}"/>
-      </geometry>
-    </collision>
-    <visual>
-      <origin xyz="${foot_length/2-down_width/2} ${foot_width/2} ${-foot_height/2}" rpy="0 0 0"/>
-      <geometry>
-	    <box size="${foot_length} ${foot_width} ${foot_height}"/>
-      </geometry>
-      <material name="orange"/>
-    </visual>
-    <inertial>
-      <origin xyz="${foot_length/2-down_width/2} ${foot_width/2} ${-foot_height/2}" rpy="0 0 0"/>
-      <mass value="${foot_mass}"/>
-      <inertia
-	  ixx="${foot_mass / 12.0 * (foot_width*foot_width + foot_height*foot_height)}" ixy="0.0" ixz="0.0"
-	  iyy="${foot_mass / 12.0 * (foot_length*foot_length + foot_height*foot_height)}" iyz="0.0"
-	  izz="${foot_mass / 12.0 * (foot_length*foot_length + foot_width*foot_width)}"/>
+      <origin xyz="${foot_back_length/2-down_width/2} ${foot_width/2} ${-foot_height/2}" rpy="0 0 0"/>
+      <geometry>
+	    <box size="${foot_back_length} ${foot_width} ${foot_height}"/>
+      </geometry>
+    </collision>
+    <visual>
+      <origin xyz="${foot_back_length/2-down_width/2} ${foot_width/2} ${-foot_height/2}" rpy="0 0 0"/>
+      <geometry>
+	    <box size="${foot_back_length} ${foot_width} ${foot_height}"/>
+      </geometry>
+      <material name="orange"/>
+    </visual>
+    <inertial>
+      <origin xyz="${foot_back_length/2-down_width/2} ${foot_width/2} ${-foot_height/2}" rpy="0 0 0"/>
+      <mass value="${foot_back_mass}"/>
+      <inertia
+	  ixx="${foot_back_mass / 12.0 * (foot_width*foot_width + foot_height*foot_height)}" ixy="0.0" ixz="0.0"
+	  iyy="${foot_back_mass / 12.0 * (foot_back_length*foot_back_length + foot_height*foot_height)}" iyz="0.0"
+	  izz="${foot_back_mass / 12.0 * (foot_back_length*foot_back_length + foot_width*foot_width)}"/>
+    </inertial>
+  </link>
+  <joint name="LFF_joint" type="revolute">
+    <limit
+       velocity="${foot_maxvel}" effort="${foot_effort}" lower="${foot_front_lower}" upper="${foot_front_upper}" />
+    <parent link="LF_link"/>
+    <child link="LFF_link"/>
+    <origin xyz="${foot_back_length-down_width/2} 0 0" rpy="0 0 0"/>
+    <axis xyz="0 1 0"/>
+    <dynamics damping="0.7"/>
+  </joint>
+  <link name="LFF_link">
+    <gazebo>
+        <self_collide>1</self_collide>
+    </gazebo>
+    <collision>
+      <origin xyz="${foot_front_length/2} ${-foot_width/2} ${-foot_height/2}" rpy="0 0 0"/>
+      <geometry>
+	    <box size="${foot_front_length} ${foot_width} ${foot_height}"/>
+      </geometry>
+    </collision>
+    <visual>
+      <origin xyz="${foot_front_length/2} ${-foot_width/2} ${-foot_height/2}" rpy="0 0 0"/>
+      <geometry>
+	    <box size="${foot_front_length} ${foot_width} ${foot_height}"/>
+      </geometry>
+      <material name="orange"/>
+    </visual>
+    <inertial>
+      <origin xyz="${foot_front_length/2} ${-foot_width/2} ${-foot_height/2}" rpy="0 0 0"/>
+      <mass value="${foot_front_mass}"/>
+      <inertia
+	  ixx="${foot_front_mass / 12.0 * (foot_width*foot_width + foot_height*foot_height)}" ixy="0.0" ixz="0.0"
+	  iyy="${foot_front_mass / 12.0 * (foot_front_length*foot_front_length + foot_height*foot_height)}" iyz="0.0"
+	  izz="${foot_front_mass / 12.0 * (foot_front_length*foot_front_length + foot_width*foot_width)}"/>
+    </inertial>
+  </link>
+  <joint name="RFF_joint" type="revolute">
+    <limit
+       velocity="${foot_maxvel}" effort="${foot_effort}" lower="${foot_front_lower}" upper="${foot_front_upper}" />
+    <parent link="RF_link"/>
+    <child link="RFF_link"/>
+    <origin xyz="${foot_back_length-down_width/2} 0 0" rpy="0 0 0"/>
+    <axis xyz="0 1 0"/>
+    <dynamics damping="0.7"/>
+  </joint>
+  <link name="RFF_link">
+    <gazebo>
+        <self_collide>1</self_collide>
+    </gazebo>
+    <collision>
+      <origin xyz="${foot_front_length/2} ${foot_width/2} ${-foot_height/2}" rpy="0 0 0"/>
+      <geometry>
+	    <box size="${foot_front_length} ${foot_width} ${foot_height}"/>
+      </geometry>
+    </collision>
+    <visual>
+      <origin xyz="${foot_front_length/2} ${foot_width/2} ${-foot_height/2}" rpy="0 0 0"/>
+      <geometry>
+	    <box size="${foot_front_length} ${foot_width} ${foot_height}"/>
+      </geometry>
+      <material name="orange"/>
+    </visual>
+    <inertial>
+      <origin xyz="${foot_front_length/2} ${foot_width/2} ${-foot_height/2}" rpy="0 0 0"/>
+      <mass value="${foot_front_mass}"/>
+      <inertia
+	  ixx="${foot_front_mass / 12.0 * (foot_width*foot_width + foot_height*foot_height)}" ixy="0.0" ixz="0.0"
+	  iyy="${foot_front_mass / 12.0 * (foot_front_length*foot_front_length + foot_height*foot_height)}" iyz="0.0"
+	  izz="${foot_front_mass / 12.0 * (foot_front_length*foot_front_length + foot_width*foot_width)}"/>
     </inertial>
   </link>

Commit message: add friction

File: urdf/robot.xacro (robot description, xacro)
@@ -3,10 +3,10 @@
   <xacro:property name="PI" value="3.1415926535897931"/>
   <!--waist property-->
-  <xacro:property name="waist_mass" value="5" />
+  <xacro:property name="waist_mass" value="10" />
   <xacro:property name="waist_length" value="0.45" />
   <xacro:property name="waist_width" value="0.15" />
   <xacro:property name="waist_height" value="0.05" />
   <!--up property-->
-  <xacro:property name="up_mass" value="6" />
+  <xacro:property name="up_mass" value="8" />
   <xacro:property name="up_length" value="0.5" />
   <xacro:property name="up_width" value="0.1" />
@@ -17,5 +17,5 @@
   <xacro:property name="up_maxvel" value="${2*PI}" />
   <!--down property-->
-  <xacro:property name="down_mass" value="4" />
+  <xacro:property name="down_mass" value="3" />
   <xacro:property name="down_length" value="0.5" />
   <xacro:property name="down_width" value="0.1" />
@@ -26,5 +26,5 @@
   <xacro:property name="down_maxvel" value="${PI*3}" />
   <!--foot property-->
-  <xacro:property name="foot_back_mass" value="0.5" />
+  <xacro:property name="foot_back_mass" value="1" />
   <xacro:property name="foot_front_mass" value="0.5" />
   <xacro:property name="foot_back_length" value="0.15" />
